File: hardware/arduino-doorbell/arduino-doorbell.sch (EAGLE design)
At the start: 8 parts, among them T1 BC337

Commit message: Eagle Schematic update
Parts:
- removed C2: 220u, rcl:C-EU050-025X075
- added C3: 470uF, rcl:CPOL-EUE3.5-10
- added C4: 4u7, rcl:CPOL-EUE3.5-10
- added C5: 10nF, rcl:C-EU025-030X050
- added C6: 47uF, rcl:CPOL-EUE3.5-10
- added D2: MBRA340T3, diode:MBRA340T3
- added IC1: TPS5410, texas:TPS5410
- added L1: 68uF, inductor-coilcraft:DO3316P
- added R10, R12, R14, R4, R6, R7: 10k, rcl:R-EU_0204/5
- added R11: 1k13, rcl:R-EU_0204/5
- added R13: 200, rcl:R-EU_0204/5
- added R15: 10, rcl:R-EU_0204/5
- added R16, R17: 220, rcl:R-EU_0204/5
- added R5: 2k, rcl:R-EU_0204/5
- added R8, R9: 1k, rcl:R-EU_0204/5
- added T2, T3: (no value), transistor:-PNP-TO92
- added T4, T5: (no value), transistor:-NPN-SOT23-EBC
Connections:
- new net +27V: C1.2, C3.+, C4.+, IC1.VIN, R3.2
- new net GND: C3.-, C4.-, C6.-, D2.A, IC1.GND, R11.1, R12.1, R14.1, R5.1, R6.1, R8.1, R9.1, T4.E, T5.E, X1-1.1
- new net IN_C: R9.2, T3.C
- new net IN_D: R8.2, T2.C
- new net N$10: C5.2, D2.C, IC1.BOOT, L1.1
- new net N$11: IC1.VSENSE, R10.1, R11.2
- new net N$14: R12.2, R16.2, T4.B
- new net N$15: R13.1, T4.C
- new net N$16: R14.2, R17.2, T5.B
- new net N$17: R15.1, T5.C
- new net N$7: R6.2, R7.1, T3.B
- new net OUT_C: R16.1
- new net OUT_D: R17.1
- new net VCC: C6.+, L1.2, R10.2, T2.E, T3.E
- new net X1: D1.A, R13.2, R15.2, R4.2, R7.2, X1-2.1
- net N$3: now also R4.1, R5.2, T2.B; no longer C1.2, C2.2, R3.2
- net N$5: now also IC1.ENA; no longer C2.1, X1-1.1
- net N$6: now also C5.1, IC1.PH; no longer D1.A, X1-2.1
