File: hardware/interface-pcb/bus_data.kicad_sch (KiCad schematic)
At the start: 24 parts, among them Q3 BCP56-16, Q4 BCP56-16, U2 LM393

Commit message: Redraw the schematic with wires
The generated draft connected everything through net labels. The redraw
wires each block so the signal paths, dividers, filters and feedback
loops can be read at a glance, with a note per block on what to measure
there. The ESP32 moves onto the root sheet, next to a map of the circuit
sheets and their test points.

The connectivity is unchanged: the exported netlist has the same 101
parts with the same values, footprints, LCSC numbers and population, and
the same pins on all 75 nets. PCB.md describes the new layout of the
sheets and what to probe where, and flags two checks for the bring-up:
the DAC still reaches the current sink while TX_EN is low, and the
comparator input range.

PDF exports go to output/, which git ignores.

Co-Authored-By: Claude Opus 5.5 <noreply@anthropic.com>
Connections:
- net BIT_B: no longer names the net of Q4.1 (B), R24.2, R25.1
- net BIT_C: no longer names the net of Q4.2 (C), R23.2
- net CARRIER_B: no longer names the net of Q3.1 (B), R21.2, R22.1
- net CARRIER_C: no longer names the net of Q3.2 (C), R20.2
Other:
- note added: "03 / Bus data in and out"
- note added: "1 W"
- note added: "ACKNOWLEDGE THRESHOLD"
- note added: "BUS SENSE / 21"
- note added: "Bus sensing above | controlled pull-down stages below | comparator outputs are active low"
- note added: "CARRIER PULL-DOWN"
- note added: "COMPARATOR SUPPLY"
- note added: "DATA THRESHOLD"
- note added: "Firmware: both stages OFF at reset and on timeout. Do not leave a pull-down enabled on the idle bus."
- note added: "GPIO16: carrier for the whole telegram. GPIO17: additional pull-down for each zero bit. Values and transistor stress need load measurements."
- note added: "Probe TP7 together with TP1. R10 / R11 set the scaling; C10 filters RF. Check LM393 input common-mode margin."
- note added: "TP5 / GPIO34 Nominal threshold about 4.3 V at BUS. Measure both edges to set hysteresis."
- note added: "TP6 / GPIO35 Nominal threshold about 12.2 V at BUS. Capture the end of the telegram."
- note added: "ZERO-BIT PULL-DOWN"
- note removed: "BUS / 21 to the comparators (32 V -> 1.5 V, inside the LM393's input range at 3.3 V). Outputs are inverted: low while the bus is above the threshold. Thresholds about 4.3 V (data) and 12.2 V (acknowledge), hysteresis about 0.65 V at the bus. ALL VALUES PROVISIONAL until the scope measurement."
- note removed: "Data in"
- note removed: "Data out"
- note removed: "Test points"
- note removed: "The Arduino recipe: 200 R across the bus for the whole telegram (carrier), 10 R during each 0 bit. The base pull-downs keep both off while the ESP32 boots. The firmware must never leave them on: on an idle bus R20 alone would draw 140 mA."
- title: Siedle gateway interface board: Bus data in and out -> 03  /  Bus data in and out
- moved on the sheet: C10, C11, Q3, Q4, R10, R11, R12, R13, R14, R15, R16, R17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
