File: hardware/interface-pcb/bus_data.kicad_sch (KiCad schematic)
At the start: 24 parts, among them Q3 BCP56-16, Q4 BCP56-16, U2 LM393

Commit message: Keep the comparator inputs inside the LM393's range
The LM393's inputs work up to VCC - 2 V over its full temperature
range, 1.3 V on 3.3 V. Dividing the bus by 21 put the bus-sense input
at 1.33 V on an idle 28 V bus and 1.52 V while ringing at 32 V. The
output stays correct as long as the other input is in range, but that
leaves no margin.

R10 goes from 200 k to 330 k: the bus divided by 34 stays below
0.95 V at 32 V and below 1.3 V up to about 44 V. The references follow
(R12 240 k, R15 82 k), so the thresholds with hysteresis become about
5.5 V rising and 4.5 V falling for data, 13.1 V and 12.1 V for the
acknowledge. Still provisional until the scope measurement.

Co-Authored-By: Claude Opus 5.5 <noreply@anthropic.com>
Parts:
- R10: value 200k -> 330k
- R12: value 150k -> 240k
- R15: value 47k -> 82k
Other:
- note added: "BUS SENSE / 34"
- note added: "Probe TP7 together with TP1. R10 / R11 set the scaling; C10 filters RF. 32 V -> 0.94 V, inside the LM393 input range."
- note added: "TP5 / GPIO34 Threshold about 5.5 V rising, 4.5 V falling. Measure both edges to set hysteresis."
- note added: "TP6 / GPIO35 Threshold about 13.1 V rising, 12.1 V falling. Capture the end of the telegram."
- note removed: "BUS SENSE / 21"
- note removed: "Probe TP7 together with TP1. R10 / R11 set the scaling; C10 filters RF. Check LM393 input common-mode margin."
- note removed: "TP5 / GPIO34 Nominal threshold about 4.3 V at BUS. Measure both edges to set hysteresis."
- note removed: "TP6 / GPIO35 Nominal threshold about 12.2 V at BUS. Capture the end of the telegram."
Changed lines of the file:
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@@
 		)
 	)
-	(text "BUS SENSE / 21"
+	(text "BUS SENSE / 34"
 		(exclude_from_sim no)
 		(at 17.78 50.8 0)
@@
 			)
 		)
-		(property "Value" "200k"
+		(property "Value" "330k"
 			(at 46.99 90.551 0)
 			(show_name no)
@@
 			)
 		)
-		(property "Value" "150k"
+		(property "Value" "240k"
 			(at 140.97 85.471 0)
 			(show_name no)
@@
 			)
 		)
-		(property "Value" "47k"
+		(property "Value" "82k"
 			(at 280.67 85.471 0)
 			(show_name no)
@@
 		)
 	)
-	(text "Probe TP7 together with TP1.\nR10 / R11 set the scaling; C10 filters RF.\nCheck LM393 input common-mode margin."
+	(text "Probe TP7 together with TP1.\nR10 / R11 set the scaling; C10 filters RF.\n32 V -> 0.94 V, inside the LM393 input range."
 		(exclude_from_sim no)
 		(at 17.78 160.02 0)
@@
 		)
 	)
-	(text "TP5 / GPIO34\nNominal threshold about 4.3 V at BUS.\nMeasure both edges to set hysteresis."
+	(text "TP5 / GPIO34\nThreshold about 5.5 V rising, 4.5 V falling.\nMeasure both edges to set hysteresis."
 		(exclude_from_sim no)
 		(at 121.92 160.02 0)
@@
 		)
 	)
-	(text "TP6 / GPIO35\nNominal threshold about 12.2 V at BUS.\nCapture the end of the telegram."
+	(text "TP6 / GPIO35\nThreshold about 13.1 V rising, 12.1 V falling.\nCapture the end of the telegram."
 		(exclude_from_sim no)
 		(at 256.54 160.02 0)
