File: hardware/interface-pcb/bus_power.kicad_sch (KiCad schematic)
At the start: 26 parts, among them J1 Siedle bus Ta/Tb, J2 ext. 5V, Q1 IRFR120N, Q2 BC846B, U1 R-78CK5.0-0.5

Commit message: Redraw the schematic with wires
The generated draft connected everything through net labels. The redraw
wires each block so the signal paths, dividers, filters and feedback
loops can be read at a glance, with a note per block on what to measure
there. The ESP32 moves onto the root sheet, next to a map of the circuit
sheets and their test points.

The connectivity is unchanged: the exported netlist has the same 101
parts with the same values, footprints, LCSC numbers and population, and
the same pins on all 75 nets. PCB.md describes the new layout of the
sheets and what to probe where, and flags two checks for the bring-up:
the DAC still reaches the current sink while TX_EN is low, and the
comparator input range.

PDF exports go to output/, which git ignores.

Co-Authored-By: Claude Opus 5.5 <noreply@anthropic.com>
Connections:
- net +5V_BUS: no longer names the net of C5.1, JP1.1 (A), U1.3 (VOUT)
- net 5V_SEL: no longer names the net of D2.2 (A), JP1.2 (B)
- net TA: no longer names the net of F1.1, J1.1 (Pin_1)
Other:
- note added: "02 / Bus input and power"
- note added: "5 V SUPPLY"
- note added: "BENCH CHECK / TP1: bus voltage | TP2: startup, ripple, frame hold-up | TP3: 5 V rail | TP4: board GND (Tb)"
- note added: "BUS CONNECTION"
- note added: "C2 / C3 bridge data frames and Wi-Fi bursts. VOUT: about 20 V in the load simulation. U1 input range: 6.5-40 V."
- note added: "ENERGY STORAGE"
- note added: "EXTERNAL SUPPLY OPTION"
- note added: "F1: 100 mA hold BUS feeds data and audio before D1."
- note added: "GPIO36 / ADC1 VMON = VOUT / 11 Enable Wi-Fi after VOUT > about 14 V. Check threshold and recovery under load."
- note added: "GYRATOR / GATE FILTER AND CURRENT LIMIT"
- note added: "Gyrator: slow gate tracking, high AC impedance. R1 x C1 = 2.2 s; Q2 / R2 limit to about 55 mA. Confirm startup and heat on the bench."
- note added: "J2 not fitted by default. Check D1 Mini USB / 5 V power sharing before using concurrent supplies."
- note added: "JP1: cut for external power. D2 blocks reverse feed into U1."
- note added: "Ta (+)"
- note added: "Ta / Tb -> protection -> gyrator and energy storage -> 5 V supply"
- note added: "Tb (-)"
- note added: "VOUT MONITOR / WIFI START"
- note removed: "Bus input"
- note removed: "Filter and 5 V"
- note removed: "Gyrator"
- note removed: "Q1 follows the gate voltage filtered by R1/C1 (about 2 s), so the stage draws a steady current and looks like a large inductor to the bus. Q2/R2 limit the current to about 55 mA. Values from the simulation (hardware/bus-power/gyrator.cir), to be confirmed on the breadboard."
- note removed: "Ta is +, Tb is - and board ground. F1 protects the building's bus from faults on our side, TVS1 clamps surges. Data, receive and send circuits connect to BUS, before D1 (doc/Bus-Power.md)."
- note removed: "Test points and power flags"
- note removed: "Two-stage RC filter: the capacitors deliver the Wi-Fi bursts and bridge 65 ms data frames. U1 takes 6.5-40 V. D2 keeps a USB cable on the D1 Mini from feeding back into U1. Cut JP1 to run the board from J2 (external 5 V) only."
- note removed: "VOUT / 11 to GPIO36 (ADC1). The firmware starts Wi-Fi only above about 14 V, or the stage stalls (doc/Bus-Power.md)."
- note removed: "VOUT monitor"
- title: Siedle gateway interface board: Bus input and power -> 02  /  Bus input and power
- moved on the sheet: C1, C2, C3, C4, C5, D1, D2, DZ1, F1, J1, J2, JP1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
