File: hardware/interface-pcb/bus_power.kicad_sch (KiCad schematic)
At the start: 26 parts, among them J1 Siedle bus Ta/Tb, J2 ext. 5V, Q1 IRFR120N, Q2 BC846B, U1 R-78CK5.0-0.5

Commit message: Lay the 2200 uF capacitors flat on the board
Standing up, C2 and C3 are 30 mm tall and set the depth of the
wall-mounted case. Lying down, with the leads bent at the body, they
are 16 mm, about as high as the D1 Mini on its sockets.

The project footprint keeps KiCad's 16 mm / 7.5 mm pads, stacked at
one end, and gives the courtyard the whole body, so nothing gets
placed underneath. Its 3D model is KiCad's radial capacitor, turned on
its side and stretched to the 30 mm part.

Co-Authored-By: Claude Opus 5.5 <noreply@anthropic.com>
Parts:
- C2, C3: footprint Capacitor_THT:CP_Radial_D16.0mm_P7.50mm -> gateway:CP_Radial_D16.0mm_P7.50mm_Lying
Changed lines of the file:
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@@
 			)
 		)
-		(property "Footprint" "Capacitor_THT:CP_Radial_D16.0mm_P7.50mm"
+		(property "Footprint" "gateway:CP_Radial_D16.0mm_P7.50mm_Lying"
 			(at 238.76 119.38 0)
 			(hide yes)
@@
 			)
 		)
-		(property "Footprint" "Capacitor_THT:CP_Radial_D16.0mm_P7.50mm"
+		(property "Footprint" "gateway:CP_Radial_D16.0mm_P7.50mm_Lying"
 			(at 276.86 119.38 0)
 			(hide yes)

Commit message: Decouple U1's input next to its pins
The routing moved U1 to the right edge, away from the codec, which
leaves it about 32 mm from C3, its only input capacitor. A switching
regulator wants the pulsed input current supplied right at its pins,
not through a long track.

C6, a 2.2 uF / 100 V X7R in 1210, sits under the VOUT track a few
millimetres from U1's VIN, with a ground via at its GND pad. It is the
same part as C1 (C153036), so JLCPCB adds no loading fee.

Co-Authored-By: Claude Opus 5.5 <noreply@anthropic.com>
Parts:
- added C6: 2.2u 100V, Capacitor_SMD:C_1210_3225Metric, symbol Device:C
Connections:
- net GND: now also C6.2
- net VOUT: now also C6.1
Changed lines of the file:
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@@
 	)
 	(symbol
+		(lib_id "Device:C")
+		(at 297.18 111.76 0)
+		(unit 1)
+		(body_style 1)
+		(exclude_from_sim no)
+		(in_bom yes)
+		(on_board yes)
+		(in_pos_files yes)
+		(dnp no)
+		(property "Reference" "C6"
+			(at 300.99 110.109 0)
+			(show_name no)
+			(do_not_autoplace no)
+			(effects
+				(font
+					(size 1.27 1.27)
+				)
+				(justify left)
+			)
+		)
+		(property "Value" "2.2u 100V"
+			(at 300.99 113.411 0)
+			(show_name no)
+			(do_not_autoplace no)
+			(effects
+				(font
+					(size 1.27 1.27)
+				)
+				(justify left)
+			)
+		)
+		(property "Footprint" "Capacitor_SMD:C_1210_3225Metric"
+			(at 297.18 111.76 0)
+			(hide yes)
+			(show_name no)
+			(do_not_autoplace no)
+			(effects
+				(font
+					(size 1.27 1.27)
+				)
+			)
+		)
+		(property "Datasheet" ""
+			(at 297.18 111.76 0)
+			(hide yes)
+			(show_name no)
+			(do_not_autoplace no)
+			(effects
+				(font
+					(size 1.27 1.27)
+				)
+			)
+		)
+		(property "Description" "Unpolarized capacitor"
+			(at 297.18 111.76 0)
+			(hide yes)
+			(show_name no)
+			(do_not_autoplace no)
+			(effects
+				(font
+					(size 1.27 1.27)
+				)
+			)
+		)
+		(property "LCSC" "C153036"
+			(at 297.18 111.76 0)
+			(hide yes)
+			(show_name no)
+			(do_not_autoplace no)
+			(effects
+				(font
+					(size 1.27 1.27)
+				)
+			)
+		)
+		(property "Note" "U1 input, next to its pins; same part as C1"
+			(at 297.18 111.76 0)
+			(hide yes)
+			(show_name no)
+			(do_not_autoplace no)
+			(effects
+				(font
+					(size 1.27 1.27)
+				)
+			)
+		)
+		(pin "1"
+		)
+		(pin "2"
+		)
+		(instances
+			(project "interface-pcb"
+				(path "/10653c94-f447-5f87-9187-3dc11d9ab931/c68f7d0d-f82b-5cdc-80ee-9955238d066b"
+					(reference "C6")
+					(unit 1)
+				)
+			)
+		)
+	)
+	(symbol
+		(lib_id "power:GND")
+		(at 297.18 127 0)
+		(unit 1)
+		(body_style 1)
+		(exclude_from_sim no)
+		(in_bom no)
+		(on_board no)
+		(in_pos_files yes)
+		(dnp no)
+		(property "Reference" "#PWR0217"
+			(at 297.18 127 0)
+			(hide yes)
+			(show_name no)
+			(do_not_autoplace no)
+			(effects
+				(font
+					(size 1.27 1.27)
+				)
+			)
+		)
+		(property "Value" "GND"
+			(at 297.18 130.81 0)
+			(show_name no)
+			(do_not_autoplace no)
+			(effects
+				(font
+					(size 1.02 1.02)
+				)
+			)
+		)
+		(property "Footprint" ""
+			(at 297.18 127 0)
+			(hide yes)
+			(show_name no)
+			(do_not_autoplace no)
+			(effects
+				(font
+					(size 1.27 1.27)
+				)
+			)
+		)
+		(property "Datasheet" ""
+			(at 297.18 127 0)
+			(hide yes)
+			(show_name no)
+			(do_not_autoplace no)
+			(effects
+				(font
+					(size 1.27 1.27)
+				)
+			)
+		)
+		(property "Description" "Power symbol creates a global label with name \"GND\" , ground"
+			(at 297.18 127 0)
+			(hide yes)
+			(show_name no)
+			(do_not_autoplace no)
+			(effects
+				(font
+					(size 1.27 1.27)
+				)
+			)
+		)
+		(pin "1"
+		)
+		(instances
+			(project "interface-pcb"
+				(path "/10653c94-f447-5f87-9187-3dc11d9ab931/c68f7d0d-f82b-5cdc-80ee-9955238d066b"
+					(reference "#PWR0217")
+					(unit 1)
+				)
+			)
+		)
+	)
+	(symbol
 		(lib_id "Connector:Screw_Terminal_01x02")
 		(at 25.4 86.36 0)
@@
 		(pts
 			(xy 287.02 86.36)
+			(xy 297.18 86.36)
+		)
+		(stroke
+			(width 0)
+			(type default)
+		)
+	)
+	(wire
+		(pts
+			(xy 297.18 86.36)
 			(xy 304.8 86.36)
 		)
@@
 	(wire
 		(pts
+			(xy 297.18 86.36)
+			(xy 297.18 107.95)
+		)
+		(stroke
+			(width 0)
+			(type default)
+		)
+	)
+	(wire
+		(pts
+			(xy 297.18 115.57)
+			(xy 297.18 127)
+		)
+		(stroke
+			(width 0)
+			(type default)
+		)
+	)
+	(wire
+		(pts
 			(xy 314.96 96.52)
 			(xy 314.96 127)
@@
 	)
 	(junction
+		(at 297.18 86.36)
+		(diameter 0)
+		(color 0 0 0 0)
+	)
+	(junction

Commit message: Use 1000 uF / 35 V for C2 and C3
The 2200 uF / 50 V capacitors were the tallest parts after the D1 Mini.
Without load they sit about 4 V below the bus, 28 V while it rings at
32 V, so 35 V parts are enough; and smaller capacitors filter the Wi-Fi
bursts as well when R3 and R4 grow with them. C2 and C3 become
1000 uF / 35 V (13 x 20 mm, LCSC C10749), R3 and R4 33 and 39 ohms.

The decision comes before the bus measurements on purpose: if the bus
rings above 32 V, the 2200 uF / 50 V parts with 15 and 18 ohms go back
in, and the 16 mm footprint and model stay in the library for that.

Both variants get the change. A new lying footprint (5 mm pitch) and its
3D model replace the 16 mm ones on the boards; pad 1 stays put, pad 2
moves 2.5 mm closer and lands on C3's VOUT feed, which now runs straight
down to pad 1's track. gyrator.cir takes the new values: 3.2 s to 14 V,
VOUT 19.2 V, a 0.83 V dip during a frame, 130-170 kohm toward the bus
at speech frequencies.

ERC: no violations in both projects. DRC with schematic parity on the
D1 Mini board: 0 violations, 0 unconnected items, 0 parity issues. The
S3 board shows only the parity issues of its pending layout.

Co-Authored-By: Claude Opus 5.5 <noreply@anthropic.com>
Parts:
- C2: value 2200u 50V -> 1000u 35V; footprint gateway:CP_Radial_D16.0mm_P7.50mm_Lying -> gateway:CP_Radial_D13.0mm_P5.00mm_Lying; LCSC C13917 -> C10749; Note 16 x 30 mm, lay down; hand-soldered -> 13 x 20 mm, lying; hand-soldered
- C3: value 2200u 50V -> 1000u 35V; footprint gateway:CP_Radial_D16.0mm_P7.50mm_Lying -> gateway:CP_Radial_D13.0mm_P5.00mm_Lying; LCSC C13917 -> C10749
- R3: value 15 -> 33; LCSC C17480 -> C17634
- R4: value 18 -> 39; LCSC C17507 -> (none)
Changed lines of the file:
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@@
 			)
 		)
-		(property "Value" "15"
+		(property "Value" "33"
 			(at 220.98 83.312 90)
 			(show_name no)
@@
 			)
 		)
-		(property "LCSC" "C17480"
+		(property "LCSC" "C17634"
 			(at 220.98 86.36 0)
 			(hide yes)
@@
 			)
 		)
-		(property "Value" "2200u 50V"
+		(property "Value" "1000u 35V"
 			(at 242.57 121.031 0)
 			(show_name no)
@@
 			)
 		)
-		(property "Footprint" "gateway:CP_Radial_D16.0mm_P7.50mm_Lying"
+		(property "Footprint" "gateway:CP_Radial_D13.0mm_P5.00mm_Lying"
 			(at 238.76 119.38 0)
 			(hide yes)
@@
 			)
 		)
-		(property "LCSC" "C13917"
+		(property "LCSC" "C10749"
 			(at 238.76 119.38 0)
 			(hide yes)
@@
 			)
 		)
-		(property "Note" "16 x 30 mm, lay down; hand-soldered"
+		(property "Note" "13 x 20 mm, lying; hand-soldered"
 			(at 238.76 119.38 0)
 			(hide yes)
@@
 			)
 		)
-		(property "Value" "18"
+		(property "Value" "39"
 			(at 256.54 83.312 90)
 			(show_name no)
@@
 			)
 		)
-		(property "LCSC" "C17507"
+		(property "LCSC" ""
 			(at 256.54 86.36 0)
 			(hide yes)
@@
 			)
 		)
-		(property "Value" "2200u 50V"
+		(property "Value" "1000u 35V"
 			(at 280.67 121.031 0)
 			(show_name no)
@@
 			)
 		)
-		(property "Footprint" "gateway:CP_Radial_D16.0mm_P7.50mm_Lying"
+		(property "Footprint" "gateway:CP_Radial_D13.0mm_P5.00mm_Lying"
 			(at 276.86 119.38 0)
 			(hide yes)
@@
 			)
 		)
-		(property "LCSC" "C13917"
+		(property "LCSC" "C10749"
 			(at 276.86 119.38 0)
 			(hide yes)
