File: hardware/interface-pcb/audio.kicad_sch (KiCad schematic)
At the start: 40 parts, among them Q5 BC846B, U3 ES8311, U4 MCP6002

Commit message: Redraw the schematic with wires
The generated draft connected everything through net labels. The redraw
wires each block so the signal paths, dividers, filters and feedback
loops can be read at a glance, with a note per block on what to measure
there. The ESP32 moves onto the root sheet, next to a map of the circuit
sheets and their test points.

The connectivity is unchanged: the exported netlist has the same 101
parts with the same values, footprints, LCSC numbers and population, and
the same pins on all 75 nets. PCB.md describes the new layout of the
sheets and what to probe where, and flags two checks for the bring-up:
the DAC still reaches the current sink while TX_EN is low, and the
comparator input range.

PDF exports go to output/, which git ignores.

Co-Authored-By: Claude Opus 5.5 <noreply@anthropic.com>
Connections:
- net MIC1N: no longer names the net of C40.1, U3.17 (MIC1N)
- net RX_AC: no longer names the net of C37.2, R34.1
- net RX_BUS: no longer names the net of C37.1, JP2.2 (B)
- net TX_B: no longer names the net of Q5.1 (B), R40.2
- net TX_BUS: no longer names the net of JP3.1 (A), R41.2
- net TX_C: no longer names the net of Q5.3 (C), R41.1
- net U4B_OUT: no longer names the net of U4.6 (-), U4.7
Other:
- note added: "04 / Audio codec and bus interface"
- note added: "BUS RECEIVE / AC COUPLING"
- note added: "BUS TRANSMIT / BIAS AND CURRENT FEEDBACK"
- note added: "CODEC / ES8311"
- note added: "I2C address: 0x18 (CE low). R30 fitted: MCLK held low; select SCLK in codec registers. R31 DNP: optional GPIO0 MCLK, remove R30 first."
- note added: "I2S and I2C connect to the controller | receive and transmit share BUS | gains remain provisional"
- note added: "JP2: cut to disconnect receive from BUS. TP8: speech amplitude and telegram-step recovery. Set attenuation / codec gain from measured speech."
- note added: "JP3: cut to isolate the current sink. TP9: DC bias, speech swing and clipping. Verify the off state with the DAC active."
- note added: "OP-AMP SUPPLY / UNUSED HALF"
- note added: "TX_EN: GPIO4, ramp the bias. I(Q5) is approximately V(TX_FB) / R42. Set current and gain after measuring bus impedance."
- note removed: "C37 blocks the bus DC. R34 and the BAT54S clamps catch the ~26 V steps of every telegram. R35/R36 bias the node at mid-rail. Speech divides by about 0.56 into the codec's 6 k input; the PGA sets the gain. High-pass ~150 Hz. Cut JP2 to take the receive path off the bus."
- note removed: "Codec"
- note removed: "Current sink: the bus current through Q5 follows the voltage at TX_SUM divided by R42. TX_EN (GPIO4) ramps a DC bias of about 2.8 mA up over ~0.1 s, the DAC adds the speech on top. Off while TX_EN is low. Values provisional until the bus impedance is measured. Cut JP3 to take the stage off the bus."
- note removed: "ES8311 at I2C address 0x18 (CE low). Master clock from the I2S bit clock by default (R30 fitted); for a real MCLK swap R30 for R31 (GPIO0, the only MCLK pin of the classic ESP32). Placed by the board house."
- note removed: "Receive"
- note removed: "Send"
- note removed: "Test points"
- title: Siedle gateway interface board: Audio -> 04  /  Audio codec and bus interface
- moved on the sheet: C30, C31, C32, C33, C34, C35, C36, C37, C38, C39, C40, C41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

Commit message: Name the MIC1N net
The redraw wired MIC1N directly, so the Codec net class matched it by
KiCad's pin-derived name, Net-(U3-MIC1N), which changes when U3 or
its pins are renumbered. A label makes it /Audio/MIC1N in the
schematic, the board and the net class pattern.

Co-Authored-By: Claude Opus 5.5 <noreply@anthropic.com>
Connections:
- net MIC1N: now reaches C40.1, U3.17 (MIC1N)
Changed lines of the file:
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@@
+		)
+	)
+	(label "MIC1N"
+		(at 175.26 124.46 90)
+		(effects
+			(font
+				(size 1.27 1.27)
+			)
+			(justify left bottom)
 		)
 	)
