File: hardware/interface-pcb/interface-pcb.kicad_pcb (KiCad board)
At the start: 2 copper layers, 90 x 75 mm, 102 parts, among them J1 Siedle bus Ta/Tb, J2 ext. 5V, Q1 IRFR120N, Q2 BC846B, Q3 BCP56-16, Q4 BCP56-16, Q5 BC846B, SW1 setup, U1 R-78CK5.0-0.5, U2 LM393, U3 ES8311, U4 MCP6002, U5 ESP32 D1 Mini

Commit message: Tighten the codec's receive node and VMID capacitor
RX_IN, the node after R34 that the bias resistors hold at mid-rail
through 50 k, is the most sensitive net on the board: it picks up
whatever couples into it. It ran 40 mm over both layers, because R35,
R36 and TP8 sat at the top of the codec area, away from the clamp
diodes and the coupling capacitor. C34, VMID's filter capacitor, sat
6.9 mm from its pin.

R35 and R36 move into C34's old place next to D30, TP8 next to C39,
and C34 under U3's VMID pin. RX_IN, VMID, ADCVREF and the local +3V3
branch were ripped up and rerouted with Freerouting, with all other
copper locked; only the new tracks were carried over. RX_IN is now
24 mm on the top layer without vias, VMID 2.5 mm. A stitching via
reconnects the ground island around C34; labels moved to clear.

DRC with refilled zones: no violations, no unconnected items, no
schematic parity issues.

Co-Authored-By: Claude Opus 5.5 <noreply@anthropic.com>
Parts:
- moved TP8 22.6 mm to (89.6, 104.0)
- moved R36 13.2 mm to (80.6, 105.0), turned to 180 degrees
- moved R35 12.0 mm to (80.6, 103.0)
- moved C34 4.61 mm to (83.3, 100.0)
Routing:
- net /Audio/RX_IN: track 40.1 -> 24.0 mm, vias 2 -> 0
- net +3V3: track 185.0 -> 172.0 mm, vias 7 -> 5
- net /Audio/VMID: track 7.43 -> 2.47 mm
