File: hardware/interface-pcb-s3/audio.kicad_sch (KiCad schematic)
At the start: 40 parts, among them Q5 BC846B, U3 ES8311, U4 MCP6002

Commit message: Put an ESP32-S3 module on the board and run it on 3.3 V
The S3 variant replaces the plug-in D1 Mini with an ESP32-S3-WROOM-1-
N16R8 that JLCPCB places (C2913202). That saves the second board
revision that was planned for a module, and the 8 MB PSRAM runs ESP-SR's
echo cancellation for full duplex.

Without the D1 Mini nothing needs 5 V: U1 becomes the R-78CK3.3-0.5 and
feeds the module, the codec, the comparators and the op-amp directly,
instead of losing a third in the D1 Mini's linear regulator. JP1 goes;
D2 now feeds the unfitted J2 (9-24 V) into VOUT ahead of U1, where the
gyrator steps back by itself.

The controller sheet gets the module with its decoupling and power-on
reset (EN 10 k / 1 uF, SW2), USB-C on the S3's native USB for flashing
and logs (USBLC6 ESD protection, 5.1 k CC pull-downs, VBUS not used for
power), UART0 test points, and SW1 moves to GPIO0, the BOOT pin the
firmware already uses for the setup hotspot. PCB-S3.md has the pin plan
and the differences against the D1 Mini variant.

ERC: no violations. Compared with the D1 Mini variant's netlist, only
the supply, the module and the new parts changed. The layout still
shows the D1 Mini; it follows after the review.

Co-Authored-By: Claude Opus 5.5 <noreply@anthropic.com>
Connections:
- net +5V is gone; now on net +3V3: C44.1, U4.8 (V+)
Other:
- note added: "I2C address: 0x18 (CE low). R30 fitted: MCLK held low; select SCLK in codec registers. R31 DNP: optional MCLK from GPIO10, remove R30 first."
- note added: "TX_EN: GPIO15, ramp the bias. I(Q5) is approximately V(TX_FB) / R42. Set current and gain after measuring bus impedance."
- note removed: "I2C address: 0x18 (CE low). R30 fitted: MCLK held low; select SCLK in codec registers. R31 DNP: optional GPIO0 MCLK, remove R30 first."
- note removed: "TX_EN: GPIO4, ramp the bias. I(Q5) is approximately V(TX_FB) / R42. Set current and gain after measuring bus impedance."
Changed lines of the file:
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@@
 		)
 	)
-	(text "I2C address: 0x18 (CE low).\nR30 fitted: MCLK held low; select SCLK in codec registers.\nR31 DNP: optional GPIO0 MCLK, remove R30 first."
+	(text "I2C address: 0x18 (CE low).\nR30 fitted: MCLK held low; select SCLK in codec registers.\nR31 DNP: optional MCLK from GPIO10, remove R30 first."
 		(exclude_from_sim no)
 		(at 17.78 127 0)
@@
 	)
 	(symbol
-		(lib_id "power:+5V")
+		(lib_id "power:+3V3")
 		(at 302.26 203.2 0)
 		(unit 1)
@@
 			)
 		)
-		(property "Value" "+5V"
+		(property "Value" "+3V3"
 			(at 302.26 199.39 0)
 			(show_name no)
@@
 		)
 	)
-	(text "TX_EN: GPIO4, ramp the bias.\nI(Q5) is approximately V(TX_FB) / R42.\nSet current and gain after measuring bus impedance."
+	(text "TX_EN: GPIO15, ramp the bias.\nI(Q5) is approximately V(TX_FB) / R42.\nSet current and gain after measuring bus impedance."
 		(exclude_from_sim no)
 		(at 17.78 274.32 0)
