File: hardware/interface-pcb-s3/bus_data.kicad_sch (KiCad schematic)
At the start: 24 parts, among them Q3 BCP56-16, Q4 BCP56-16, U2 LM393

Commit message: Put an ESP32-S3 module on the board and run it on 3.3 V
The S3 variant replaces the plug-in D1 Mini with an ESP32-S3-WROOM-1-
N16R8 that JLCPCB places (C2913202). That saves the second board
revision that was planned for a module, and the 8 MB PSRAM runs ESP-SR's
echo cancellation for full duplex.

Without the D1 Mini nothing needs 5 V: U1 becomes the R-78CK3.3-0.5 and
feeds the module, the codec, the comparators and the op-amp directly,
instead of losing a third in the D1 Mini's linear regulator. JP1 goes;
D2 now feeds the unfitted J2 (9-24 V) into VOUT ahead of U1, where the
gyrator steps back by itself.

The controller sheet gets the module with its decoupling and power-on
reset (EN 10 k / 1 uF, SW2), USB-C on the S3's native USB for flashing
and logs (USBLC6 ESD protection, 5.1 k CC pull-downs, VBUS not used for
power), UART0 test points, and SW1 moves to GPIO0, the BOOT pin the
firmware already uses for the setup hotspot. PCB-S3.md has the pin plan
and the differences against the D1 Mini variant.

ERC: no violations. Compared with the D1 Mini variant's netlist, only
the supply, the module and the new parts changed. The layout still
shows the D1 Mini; it follows after the review.

Co-Authored-By: Claude Opus 5.5 <noreply@anthropic.com>
Other:
- note added: "GPIO6: carrier for the whole telegram. GPIO7: additional pull-down for each zero bit. Values and transistor stress need load measurements."
- note added: "TP5 / GPIO4 Threshold about 5.5 V rising, 4.5 V falling. Measure both edges to set hysteresis."
- note added: "TP6 / GPIO5 Threshold about 13.1 V rising, 12.1 V falling. Capture the end of the telegram."
- note removed: "GPIO16: carrier for the whole telegram. GPIO17: additional pull-down for each zero bit. Values and transistor stress need load measurements."
- note removed: "TP5 / GPIO34 Threshold about 5.5 V rising, 4.5 V falling. Measure both edges to set hysteresis."
- note removed: "TP6 / GPIO35 Threshold about 13.1 V rising, 12.1 V falling. Capture the end of the telegram."
Changed lines of the file:
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@@
 		)
 	)
-	(text "TP5 / GPIO34\nThreshold about 5.5 V rising, 4.5 V falling.\nMeasure both edges to set hysteresis."
+	(text "TP5 / GPIO4\nThreshold about 5.5 V rising, 4.5 V falling.\nMeasure both edges to set hysteresis."
 		(exclude_from_sim no)
 		(at 121.92 160.02 0)
@@
 		)
 	)
-	(text "TP6 / GPIO35\nThreshold about 13.1 V rising, 12.1 V falling.\nCapture the end of the telegram."
+	(text "TP6 / GPIO5\nThreshold about 13.1 V rising, 12.1 V falling.\nCapture the end of the telegram."
 		(exclude_from_sim no)
 		(at 256.54 160.02 0)
@@
 		)
 	)
-	(text "GPIO16: carrier for the whole telegram.\nGPIO17: additional pull-down for each zero bit.\nValues and transistor stress need load measurements."
+	(text "GPIO6: carrier for the whole telegram.\nGPIO7: additional pull-down for each zero bit.\nValues and transistor stress need load measurements."
 		(exclude_from_sim no)
 		(at 17.78 266.7 0)
