File: hardware/interface-pcb-s3/bus_power.kicad_sch (KiCad schematic)
At the start: 27 parts, among them J1 Siedle bus Ta/Tb, J2 ext. 5V, Q1 IRFR120N, Q2 BC846B, U1 R-78CK5.0-0.5

Commit message: Put an ESP32-S3 module on the board and run it on 3.3 V
The S3 variant replaces the plug-in D1 Mini with an ESP32-S3-WROOM-1-
N16R8 that JLCPCB places (C2913202). That saves the second board
revision that was planned for a module, and the 8 MB PSRAM runs ESP-SR's
echo cancellation for full duplex.

Without the D1 Mini nothing needs 5 V: U1 becomes the R-78CK3.3-0.5 and
feeds the module, the codec, the comparators and the op-amp directly,
instead of losing a third in the D1 Mini's linear regulator. JP1 goes;
D2 now feeds the unfitted J2 (9-24 V) into VOUT ahead of U1, where the
gyrator steps back by itself.

The controller sheet gets the module with its decoupling and power-on
reset (EN 10 k / 1 uF, SW2), USB-C on the S3's native USB for flashing
and logs (USBLC6 ESD protection, 5.1 k CC pull-downs, VBUS not used for
power), UART0 test points, and SW1 moves to GPIO0, the BOOT pin the
firmware already uses for the setup hotspot. PCB-S3.md has the pin plan
and the differences against the D1 Mini variant.

ERC: no violations. Compared with the D1 Mini variant's netlist, only
the supply, the module and the new parts changed. The layout still
shows the D1 Mini; it follows after the review.

Co-Authored-By: Claude Opus 5.5 <noreply@anthropic.com>
Parts:
- removed JP1: bus 5V, Jumper:SolderJumper-2_P1.3mm_Bridged_RoundedPad1.0x1.5mm, symbol Jumper:SolderJumper_2_Bridged
- D2: Note (none) -> blocks the bus side from J2, and reverse polarity
- J2: value ext. 5V -> ext. 9-24V
- TP3: value 5V -> 3V3
- U1: value R-78CK5.0-0.5 -> R-78CK3.3-0.5
Connections:
- net VOUT: now also D2.1 (K)
- removed net +5V: D2.1 (K), J2.1 (Pin_1), TP3.1
- net +5V_BUS renamed +3V3
- net +3V3: now also TP3.1
- net 5V_SEL: no longer names the net of D2.2 (A)
- net 5V_SEL: now also J2.1 (Pin_1)
Other:
- note added: "3.3 V SUPPLY"
- note added: "BENCH CHECK / TP1: bus voltage | TP2: startup, ripple, frame hold-up | TP3: 3.3 V rail | TP4: board GND (Tb)"
- note added: "GPIO1 / ADC1 VMON = VOUT / 11 Enable Wi-Fi after VOUT > about 14 V. Check threshold and recovery under load."
- note added: "J2 not fitted by default: 9-24 V DC into VOUT through D2, if the bus cannot power the gateway. Isolated adapter only: board GND is Tb."
- note added: "Ta / Tb -> protection -> gyrator and energy storage -> 3.3 V supply"
- note added: "U1 feeds the ESP32-S3, the codec, the comparators and the op-amp: 3.3 V only."
- note removed: "5 V SUPPLY"
- note removed: "BENCH CHECK / TP1: bus voltage | TP2: startup, ripple, frame hold-up | TP3: 5 V rail | TP4: board GND (Tb)"
- note removed: "GPIO36 / ADC1 VMON = VOUT / 11 Enable Wi-Fi after VOUT > about 14 V. Check threshold and recovery under load."
- note removed: "J2 not fitted by default. Check D1 Mini USB / 5 V power sharing before using concurrent supplies."
- note removed: "JP1: cut for external power. D2 blocks reverse feed into U1."
- note removed: "Ta / Tb -> protection -> gyrator and energy storage -> 5 V supply"

Commit message: Use 1000 uF / 35 V for C2 and C3
The 2200 uF / 50 V capacitors were the tallest parts after the D1 Mini.
Without load they sit about 4 V below the bus, 28 V while it rings at
32 V, so 35 V parts are enough; and smaller capacitors filter the Wi-Fi
bursts as well when R3 and R4 grow with them. C2 and C3 become
1000 uF / 35 V (13 x 20 mm, LCSC C10749), R3 and R4 33 and 39 ohms.

The decision comes before the bus measurements on purpose: if the bus
rings above 32 V, the 2200 uF / 50 V parts with 15 and 18 ohms go back
in, and the 16 mm footprint and model stay in the library for that.

Both variants get the change. A new lying footprint (5 mm pitch) and its
3D model replace the 16 mm ones on the boards; pad 1 stays put, pad 2
moves 2.5 mm closer and lands on C3's VOUT feed, which now runs straight
down to pad 1's track. gyrator.cir takes the new values: 3.2 s to 14 V,
VOUT 19.2 V, a 0.83 V dip during a frame, 130-170 kohm toward the bus
at speech frequencies.

ERC: no violations in both projects. DRC with schematic parity on the
D1 Mini board: 0 violations, 0 unconnected items, 0 parity issues. The
S3 board shows only the parity issues of its pending layout.

Co-Authored-By: Claude Opus 5.5 <noreply@anthropic.com>
Parts:
- C2: value 2200u 50V -> 1000u 35V; footprint gateway:CP_Radial_D16.0mm_P7.50mm_Lying -> gateway:CP_Radial_D13.0mm_P5.00mm_Lying; LCSC C13917 -> C10749; Note 16 x 30 mm, lay down; hand-soldered -> 13 x 20 mm, lying; hand-soldered
- C3: value 2200u 50V -> 1000u 35V; footprint gateway:CP_Radial_D16.0mm_P7.50mm_Lying -> gateway:CP_Radial_D13.0mm_P5.00mm_Lying; LCSC C13917 -> C10749
- R3: value 15 -> 33; LCSC C17480 -> C17634
- R4: value 18 -> 39; LCSC C17507 -> (none)
Changed lines of the file:
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@@
 			)
 		)
-		(property "Value" "15"
+		(property "Value" "33"
 			(at 220.98 83.312 90)
 			(show_name no)
@@
 			)
 		)
-		(property "LCSC" "C17480"
+		(property "LCSC" "C17634"
 			(at 220.98 86.36 0)
 			(hide yes)
@@
 			)
 		)
-		(property "Value" "2200u 50V"
+		(property "Value" "1000u 35V"
 			(at 242.57 121.031 0)
 			(show_name no)
@@
 			)
 		)
-		(property "Footprint" "gateway:CP_Radial_D16.0mm_P7.50mm_Lying"
+		(property "Footprint" "gateway:CP_Radial_D13.0mm_P5.00mm_Lying"
 			(at 238.76 119.38 0)
 			(hide yes)
@@
 			)
 		)
-		(property "LCSC" "C13917"
+		(property "LCSC" "C10749"
 			(at 238.76 119.38 0)
 			(hide yes)
@@
 			)
 		)
-		(property "Note" "16 x 30 mm, lay down; hand-soldered"
+		(property "Note" "13 x 20 mm, lying; hand-soldered"
 			(at 238.76 119.38 0)
 			(hide yes)
@@
 			)
 		)
-		(property "Value" "18"
+		(property "Value" "39"
 			(at 256.54 83.312 90)
 			(show_name no)
@@
 			)
 		)
-		(property "LCSC" "C17507"
+		(property "LCSC" ""
 			(at 256.54 86.36 0)
 			(hide yes)
@@
 			)
 		)
-		(property "Value" "2200u 50V"
+		(property "Value" "1000u 35V"
 			(at 280.67 121.031 0)
 			(show_name no)
@@
 			)
 		)
-		(property "Footprint" "gateway:CP_Radial_D16.0mm_P7.50mm_Lying"
+		(property "Footprint" "gateway:CP_Radial_D13.0mm_P5.00mm_Lying"
 			(at 276.86 119.38 0)
 			(hide yes)
@@
 			)
 		)
-		(property "LCSC" "C13917"
+		(property "LCSC" "C10749"
 			(at 276.86 119.38 0)
 			(hide yes)

Commit message: Feed the external supply into VFILT
J2's adapter went through D2 into VOUT, the node between C3 and U1.
On the S3 board that node sits next to the regulator, far from the
board edge where J2 belongs, and the long trace across the board would
cut the ground plane. VFILT, at C2 on the board's left edge, is a short
straight track away from a corner, and the adapter then also passes R4
and C3 as a filter. R4 drops 1-2 V, irrelevant at 9-24 V input.

Co-Authored-By: Claude Opus 5.5 <noreply@anthropic.com>
Connections:
- net VFILT: now also D2.1 (K)
- net VOUT: no longer D2.1 (K)
Other:
- note added: "J2 not fitted by default: 9-24 V DC into VFILT through D2, ahead of R4 and C3, if the bus cannot power the gateway. Isolated adapter only: GND is Tb."
- note removed: "J2 not fitted by default: 9-24 V DC into VOUT through D2, if the bus cannot power the gateway. Isolated adapter only: board GND is Tb."
Changed lines of the file:
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@@
 		)
 	)
-	(text "J2 not fitted by default: 9-24 V DC into VOUT\nthrough D2, if the bus cannot power the gateway.\nIsolated adapter only: board GND is Tb."
+	(text "J2 not fitted by default: 9-24 V DC into VFILT\nthrough D2, ahead of R4 and C3, if the bus cannot\npower the gateway. Isolated adapter only: GND is Tb."
 		(exclude_from_sim no)
 		(at 269.24 226.06 0)
@@
 		)
 	)
-	(label "VOUT"
+	(label "VFILT"
 		(at 256.54 226.06 90)
 		(effects
