File: hardware/interface-pcb-s3/interface-pcb-s3.kicad_pcb (KiCad board)
At the start: 2 copper layers, 90 x 75 mm, 103 parts, among them J1 Siedle bus Ta/Tb, J2 ext. 5V, Q1 IRFR120N, Q2 BC846B, Q3 BCP56-16, Q4 BCP56-16, Q5 BC846B, SW1 setup, U1 R-78CK5.0-0.5, U2 LM393, U3 ES8311, U4 MCP6002, U5 ESP32 D1 Mini

Commit message: Use 1000 uF / 35 V for C2 and C3
The 2200 uF / 50 V capacitors were the tallest parts after the D1 Mini.
Without load they sit about 4 V below the bus, 28 V while it rings at
32 V, so 35 V parts are enough; and smaller capacitors filter the Wi-Fi
bursts as well when R3 and R4 grow with them. C2 and C3 become
1000 uF / 35 V (13 x 20 mm, LCSC C10749), R3 and R4 33 and 39 ohms.

The decision comes before the bus measurements on purpose: if the bus
rings above 32 V, the 2200 uF / 50 V parts with 15 and 18 ohms go back
in, and the 16 mm footprint and model stay in the library for that.

Both variants get the change. A new lying footprint (5 mm pitch) and its
3D model replace the 16 mm ones on the boards; pad 1 stays put, pad 2
moves 2.5 mm closer and lands on C3's VOUT feed, which now runs straight
down to pad 1's track. gyrator.cir takes the new values: 3.2 s to 14 V,
VOUT 19.2 V, a 0.83 V dip during a frame, 130-170 kohm toward the bus
at speech frequencies.

ERC: no violations in both projects. DRC with schematic parity on the
D1 Mini board: 0 violations, 0 unconnected items, 0 parity issues. The
S3 board shows only the parity issues of its pending layout.

Co-Authored-By: Claude Opus 5.5 <noreply@anthropic.com>
Parts:
- C2, C3: value 2200u 50V -> 1000u 35V; footprint gateway:CP_Radial_D16.0mm_P7.50mm_Lying -> gateway:CP_Radial_D13.0mm_P5.00mm_Lying
- R3: value 15 -> 33
- R4: value 18 -> 39
Routing:
- net /Bus input and power/VOUT: track 116.5 -> 118.0 mm

Commit message: Lay out the ESP32-S3 board
New 90 x 65 mm outline with the module in the top-right corner, its
antenna flush with the top edge, and USB-C on the right edge so the
board can be flashed through the case. The bus side keeps the D1 Mini
board's arrangement; the audio section runs along the bottom, away
from the antenna and the regulator.

Routing is hybrid. By hand: the power path, BUS trunk and pull-down
collectors, 3.3 V and its decoupling, the codec's escapes and ground
necks, the I2S bundle with its test points on the bottom side, I2C,
TX_BIT and USB VBUS. Freerouting did the rest, finished in KiCad.
Ground pours on both layers with stitching vias; no bottom-layer tracks
under the audio stages.

DRC with schematic parity: no errors, no unconnected items; five
silkscreen warnings at the board edge are intended.

Co-Authored-By: Claude Opus 5.5 <noreply@anthropic.com>
Parts:
- removed JP1: bus 5V, Jumper:SolderJumper-2_P1.3mm_Bridged_RoundedPad1.0x1.5mm
- removed MK1: ESP32 D1 Mini, 3D only, gateway:D1_Mini_ESP32_Module_3D
- added C51: 22u, Capacitor_SMD:C_0805_2012Metric, F.Cu at (114.4, 65.0)
- added C52: 100n, Capacitor_SMD:C_0805_2012Metric, F.Cu at (114.4, 61.0)
- added C53: 1u, Capacitor_SMD:C_0805_2012Metric, F.Cu at (120.5, 107.0)
- added J3: USB-C, Connector_USB:USB_C_Receptacle_HRO_TYPE-C-31-M-12, F.Cu at (136.3, 94.0)
- added R52: 10k, Resistor_SMD:R_0805_2012Metric, F.Cu at (120.5, 103.0)
- added R53: 5.1k, Resistor_SMD:R_0805_2012Metric, F.Cu at (128.5, 89.5)
- added R54: 5.1k, Resistor_SMD:R_0805_2012Metric, F.Cu at (128.5, 98.5)
- added SW2: reset, Button_Switch_SMD:SW_Push_1P1T_XKB_TS-1187A, F.Cu at (126.0, 106.5)
- added TP15: TXD0, TestPoint:TestPoint_Pad_D1.5mm, F.Cu at (138.0, 59.5)
- added TP16: RXD0, TestPoint:TestPoint_Pad_D1.5mm, F.Cu at (138.0, 63.0)
- added U6: USBLC6-2SC6, Package_TO_SOT_SMD:SOT-23-6, F.Cu at (128.5, 94.0)
- J2: value ext. 5V -> ext. 9-24V
- TP10, TP11, TP12, TP13: moved to B.Cu
- TP3: value 5V -> 3V3
- U1: value R-78CK5.0-0.5 -> R-78CK3.3-0.5
- U5: value ESP32 D1 Mini -> ESP32-S3-WROOM-1-N16R8; footprint gateway:D1_Mini_ESP32_Socket -> RF_Module:ESP32-S3-WROOM-1
- moved J2 68.7 mm to (58.0, 110.3)
- moved D2 59.8 mm to (64.0, 109.0), turned to -90 degrees
- moved U1 59.2 mm to (104.5, 63.5), turned to 0 degrees
- moved C6 57.4 mm to (102.5, 68.6), turned to -90 degrees
- moved TP3 50.3 mm to (113.6, 70.0)
- moved H2 49.0 mm to (136.0, 103.0)
- moved C5 45.4 mm to (111.0, 68.0), turned to -90 degrees
- moved C3 38.5 mm to (104.5, 81.0), turned to 0 degrees
- moved TP2 37.5 mm to (100.3, 79.5)
- moved C4 35.9 mm to (110.5, 74.0)
- moved R6 35.4 mm to (110.5, 71.5)
- moved R5 35.3 mm to (106.5, 71.5)
- moved H3 25.8 mm to (78.0, 111.5)
- moved R50 23.7 mm to (128.7, 79.0)
- moved R51 19.8 mm to (133.0, 85.5)
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Connections:
- C44 pad 1: +5V -> +3V3
- C5 pad 1: /Bus input and power/+5V_BUS -> +3V3
- D2 pad 1: +5V -> /Bus input and power/VFILT
- D2 pad 2: /Bus input and power/5V_SEL -> Net-(D2-A)
- J2 pad 1: +5V -> Net-(D2-A)
- TP3 pad 1: +5V -> +3V3
- U1 pad 3: /Bus input and power/+5V_BUS -> +3V3
- U4 pad 8: +5V -> +3V3
- U5 pad 11: DATA_IN -> unconnected-(U5-IO18-Pad11)
- U5 pad 12: unconnected-(U5-IO23-Pad12) -> I2C_SDA
- U5 pad 13: unconnected-(U5-IO14-Pad13) -> /USB_DN
- U5 pad 14: unconnected-(U5-IO5-Pad14) -> /USB_DP
- U5 pad 16: +3V3 -> unconnected-(U5-IO46-Pad16)
- U5 pad 17: unconnected-(U5-IO9-Pad17) -> I2C_SCL
- U5 pad 18: unconnected-(U5-IO13-Pad18) -> I2S_DOUT
- U5 pad 19: unconnected-(U5-CMD-Pad19) -> I2S_WS
- U5 pad 2: unconnected-(U5-RST-Pad2) -> +3V3
- U5 pad 20: unconnected-(U5-IO10-Pad20) -> I2S_DIN
- U5 pad 21: unconnected-(U5-TXD-Pad21) -> I2S_BCLK
- U5 pad 22: GND -> I2S_MCLK
- U5 pad 24: I2S_DOUT -> unconnected-(U5-IO47-Pad24)
- U5 pad 25: I2C_SCL -> unconnected-(U5-IO48-Pad25)
- U5 pad 26: I2S_WS -> unconnected-(U5-IO45-Pad26)
- U5 pad 27: I2C_SDA -> /BUTTON
- U5 pad 28: I2S_DIN -> unconnected-(U5-IO35-Pad28)
- U5 pad 29: TX_BIT -> unconnected-(U5-IO36-Pad29)
- U5 pad 3: unconnected-(U5-NC-Pad3) -> /EN
- U5 pad 31: TX_CARRIER -> /LED
- U5 pad 32: TX_EN -> unconnected-(U5-IO39-Pad32)
- U5 pad 33: GND -> unconnected-(U5-IO40-Pad33)
- U5 pad 34: I2S_MCLK -> unconnected-(U5-IO41-Pad34)
- U5 pad 35: +5V -> unconnected-(U5-IO42-Pad35)
- U5 pad 36: /LED -> /RXD0
- U5 pad 37: unconnected-(U5-IO15-Pad37) -> /TXD0
- U5 pad 4: VMON -> DATA_IN
- U5 pad 40: unconnected-(U5-CLK-Pad40) -> GND
- U5 pad 5: unconnected-(U5-IO39-Pad5) -> ACK_IN
- U5 pad 6: I2S_BCLK -> TX_CARRIER
- U5 pad 7: ACK_IN -> VMON
- U5 pad 8: unconnected-(U5-IO18-Pad8) -> TX_EN
- U5 pad 9: /BUTTON -> TX_BIT
Routing:
- net +3V3: track 172.0 -> 263.2 mm, vias 5 -> 12
- net +5V: track 69.6 -> 0.00 mm, vias 2 -> 0
- net /EN: track 0.00 -> 66.5 mm, vias 0 -> 2
- net /Bus input and power/VOUT: track 118.0 -> 59.1 mm, vias 4 -> 0
- net /USB_DP: track 0.00 -> 50.9 mm, vias 0 -> 2
- net /USB_DN: track 0.00 -> 38.2 mm, vias 0 -> 2
- net /BUTTON: track 57.0 -> 19.4 mm
- net VMON: track 53.7 -> 18.3 mm, vias 1 -> 2
- net I2S_WS: track 79.1 -> 50.0 mm
- net ACK_IN: track 32.9 -> 61.4 mm, vias 1 -> 2
- net I2S_DOUT: track 77.9 -> 49.9 mm, vias 3 -> 1
- net TX_BIT: track 65.3 -> 39.5 mm, vias 3 -> 2
- net /Bus input and power/VFILT: track 22.6 -> 47.3 mm
- net I2S_DIN: track 72.9 -> 50.4 mm, vias 3 -> 1
- net /Bus input and power/GYR_G: track 39.2 -> 21.7 mm
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Other:
- board size 90 x 75 mm -> 90 x 65 mm
- board text added: "SIEDLE GATEWAY / ESP32-S3 / REV 1 DRAFT"
- board text removed: "SIEDLE GATEWAY / REV 1 DRAFT"
